File: mm_external_uart.kicad_sch (KiCad schematic)
At the start: 0 parts

Commit message: fin TP2
Parts:
- added C11: C, symbol Device:C
- added J4: Conn_01x04, symbol Connector_Generic:Conn_01x04
- added R20: 100Ω, symbol Device:R
Connections:
- new net: J4.3 (Pin_3), R20.1
- new net +BATT: C11.2, J4.2 (Pin_2)
- new net EXTERNAL_UART_RX: J4.4 (Pin_4)
- new net EXTERNAT_UART_TX: R20.2
- new net GND: C11.1, J4.1 (Pin_1)
Changed lines of the file:
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@@
 (kicad_sch (version 20230121) (generator eeschema)
   (paper "A4")
+  (wire (pts (xy 217.17 25.4) (xy 217.17 33.02))
+    (stroke (width 0) (type default))
+  )
+  (wire (pts (xy 124.46 80.01) (xy 119.38 80.01))
+    (stroke (width 0) (type default))
+  )
+  (wire (pts (xy 217.17 40.64) (xy 217.17 45.72))
+    (stroke (width 0) (type default))
+  )
+  (wire (pts (xy 139.7 83.82) (xy 147.32 83.82))
+    (stroke (width 0) (type default))
+  )
+  (wire (pts (xy 124.46 77.47) (xy 130.81 77.47))
+    (stroke (width 0) (type default))
+  )
+  (wire (pts (xy 189.23 62.23) (xy 147.32 62.23))
+    (stroke (width 0) (type default))
+  )
+  (wire (pts (xy 189.23 71.12) (xy 189.23 62.23))
+    (stroke (width 0) (type default))
+  )
+  (wire (pts (xy 147.32 62.23) (xy 147.32 69.85))
+    (stroke (width 0) (type default))
+  )
+  (wire (pts (xy 147.32 83.82) (xy 147.32 77.47))
+    (stroke (width 0) (type default))
+  )
+  (wire (pts (xy 138.43 74.93) (xy 138.43 77.47))
+    (stroke (width 0) (type default))
+  )
+  (wire (pts (xy 124.46 80.01) (xy 124.46 77.47))
+    (stroke (width 0) (type default))
+  )
+  (wire (pts (xy 147.32 74.93) (xy 138.43 74.93))
+    (stroke (width 0) (type default))
+  )
+  (wire (pts (xy 146.05 72.39) (xy 147.32 72.39))
+    (stroke (width 0) (type default))
+  )
+  (global_label "+BATT" (shape input) (at 146.05 72.39 180) (fields_autoplaced)
+    (effects (font (size 1.27 1.27)) (justify right))
+    (property "Intersheetrefs" "${INTERSHEET_REFS}" (at 137.1986 72.39 0)
+      (effects (font (size 1.27 1.27)) (justify right) hide)
+    )
+  )
+  (hierarchical_label "EXTERNAT_UART_TX" (shape output) (at 119.38 80.01 180) (fields_autoplaced)
+    (effects (font (size 1.27 1.27)) (justify right))
+  )
+  (hierarchical_label "EXTERNAL_UART_RX" (shape input) (at 139.7 83.82 180) (fields_autoplaced)
+    (effects (font (size 1.27 1.27)) (justify right))
+  )
+  (symbol (lib_id "Device:R") (at 134.62 77.47 270) (unit 1)
+    (in_bom yes) (on_board yes) (dnp no)
+    (property "Reference" "R20" (at 134.62 72.39 90)
+      (effects (font (size 1.27 1.27)))
+    )
+    (property "Value" "100Ω\n" (at 134.62 74.93 90)
+      (effects (font (size 1.27 1.27)))
+    )
+    (property "Footprint" "" (at 134.62 75.692 90)
+      (effects (font (size 1.27 1.27)) hide)
+    )
+    (property "Datasheet" "~" (at 134.62 77.47 0)
+      (effects (font (size 1.27 1.27)) hide)
+    )
+    (pin "2")
+    (pin "1")
+    (instances
+      (project "minimouse"
+        (path "/d8fa4cba-2469-4231-847f-065b6b829f44/d17bb1c7-f68a-465e-9a17-5858ef86fc30"
+          (reference "R20") (unit 1)
+        )
+      )
+    )
+  )
+  (symbol (lib_id "Device:C") (at 217.17 36.83 180) (unit 1)
+    (in_bom yes) (on_board yes) (dnp no) (fields_autoplaced)
+    (property "Reference" "C11" (at 220.98 35.56 0)
+      (effects (font (size 1.27 1.27)) (justify right))
+    )
+    (property "Value" "C" (at 220.98 38.1 0)
+      (effects (font (size 1.27 1.27)) (justify right))
+    )
+    (property "Footprint" "" (at 216.2048 33.02 0)
+      (effects (font (size 1.27 1.27)) hide)
+    )
+    (property "Datasheet" "~" (at 217.17 36.83 0)
+      (effects (font (size 1.27 1.27)) hide)
+    )
+    (pin "2")
+    (pin "1")
+    (instances
+      (project "minimouse"
+        (path "/d8fa4cba-2469-4231-847f-065b6b829f44/d17bb1c7-f68a-465e-9a17-5858ef86fc30"
+          (reference "C11") (unit 1)
+        )
+      )
+    )
+  )
+  (symbol (lib_id "power:GND") (at 189.23 71.12 0) (unit 1)
+    (in_bom yes) (on_board yes) (dnp no) (fields_autoplaced)
+    (property "Reference" "#PWR023" (at 189.23 77.47 0)
+      (effects (font (size 1.27 1.27)) hide)
+    )
+    (property "Value" "GND" (at 189.23 76.2 0)
+      (effects (font (size 1.27 1.27)))
+    )
+    (property "Footprint" "" (at 189.23 71.12 0)
+      (effects (font (size 1.27 1.27)) hide)
+    )
+    (property "Datasheet" "" (at 189.23 71.12 0)
+      (effects (font (size 1.27 1.27)) hide)
+    )
+    (pin "1")
+    (instances
+      (project "minimouse"
+        (path "/d8fa4cba-2469-4231-847f-065b6b829f44/d17bb1c7-f68a-465e-9a17-5858ef86fc30"
+          (reference "#PWR023") (unit 1)
+        )
+      )
+    )
+  )
+  (symbol (lib_id "Connector_Generic:Conn_01x04") (at 152.4 72.39 0) (unit 1)
+    (in_bom yes) (on_board yes) (dnp no) (fields_autoplaced)
+    (property "Reference" "J4" (at 154.94 72.39 0)
+      (effects (font (size 1.27 1.27)) (justify left))
+    )
+    (property "Value" "Conn_01x04" (at 154.94 74.93 0)
+      (effects (font (size 1.27 1.27)) (justify left))
+    )
+    (property "Footprint" "" (at 152.4 72.39 0)
+      (effects (font (size 1.27 1.27)) hide)
+    )
+    (property "Datasheet" "~" (at 152.4 72.39 0)
+      (effects (font (size 1.27 1.27)) hide)
+    )
+    (pin "3")
+    (pin "2")
+    (pin "4")
+    (pin "1")
+    (instances
+      (project "minimouse"
+        (path "/d8fa4cba-2469-4231-847f-065b6b829f44/d17bb1c7-f68a-465e-9a17-5858ef86fc30"
+          (reference "J4") (unit 1)
+        )
+      )
+    )
+  )
+  (symbol (lib_id "power:+BATT") (at 217.17 25.4 0) (unit 1)
+    (in_bom yes) (on_board yes) (dnp no) (fields_autoplaced)
+    (property "Reference" "#PWR025" (at 217.17 29.21 0)
+      (effects (font (size 1.27 1.27)) hide)
+    )
+    (property "Value" "+BATT" (at 217.17 20.32 0)
+      (effects (font (size 1.27 1.27)))
+    )
+    (property "Footprint" "" (at 217.17 25.4 0)
+      (effects (font (size 1.27 1.27)) hide)
+    )
+    (property "Datasheet" "" (at 217.17 25.4 0)
+      (effects (font (size 1.27 1.27)) hide)
+    )
+    (pin "1")
+    (instances
+      (project "minimouse"
+        (path "/d8fa4cba-2469-4231-847f-065b6b829f44/d17bb1c7-f68a-465e-9a17-5858ef86fc30"
+          (reference "#PWR025") (unit 1)
+        )
+      )
+    )
+  )
+  (symbol (lib_id "power:GND") (at 217.17 45.72 0) (unit 1)
+    (in_bom yes) (on_board yes) (dnp no) (fields_autoplaced)
+    (property "Reference" "#PWR026" (at 217.17 52.07 0)
+      (effects (font (size 1.27 1.27)) hide)
+    )
+    (property "Value" "GND" (at 217.17 50.8 0)
+      (effects (font (size 1.27 1.27)))
+    )
+    (property "Footprint" "" (at 217.17 45.72 0)
+      (effects (font (size 1.27 1.27)) hide)
+    )
+    (property "Datasheet" "" (at 217.17 45.72 0)
+      (effects (font (size 1.27 1.27)) hide)
+    )
+    (pin "1")
+    (instances
+      (project "minimouse"
+        (path "/d8fa4cba-2469-4231-847f-065b6b829f44/d17bb1c7-f68a-465e-9a17-5858ef86fc30"
+          (reference "#PWR026") (unit 1)
+        )
+      )
+    )
+  )
 )

Commit message: fin TP2 2
Changed lines of the file:
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@@
     (stroke (width 0) (type default))
   )
-  (wire (pts (xy 139.7 83.82) (xy 147.32 83.82))
+  (wire (pts (xy 120.65 86.36) (xy 147.32 86.36))
     (stroke (width 0) (type default))
   )
@@
     (stroke (width 0) (type default))
   )
-  (wire (pts (xy 147.32 83.82) (xy 147.32 77.47))
+  (wire (pts (xy 147.32 86.36) (xy 147.32 77.47))
     (stroke (width 0) (type default))
   )
@@
     (effects (font (size 1.27 1.27)) (justify right))
   )
-  (hierarchical_label "EXTERNAL_UART_RX" (shape input) (at 139.7 83.82 180) (fields_autoplaced)
+  (hierarchical_label "EXTERNAL_UART_RX" (shape input) (at 120.65 86.36 180) (fields_autoplaced)
     (effects (font (size 1.27 1.27)) (justify right))
   )

Commit message: Pistes
Parts:
- C14: renamed from C11; value C -> 2.2uF; footprint (none) -> Capacitor_SMD:C_0603_1608Metric
- J5: renamed from J4; footprint (none) -> Connector_PinHeader_2.54mm:PinHeader_1x04_P2.54mm_Vertical
- R19: renamed from R20; footprint (none) -> Resistor_SMD:R_0603_1608Metric
Connections:
- net EXTERNAL_UART_RX renamed EXT_UART_RX
- net EXTERNAT_UART_TX renamed EXT_UART_TX
Changed lines of the file:
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@@
+    (stroke (width 0) (type default))
+  )
+  (wire (pts (xy 142.24 64.77) (xy 142.24 72.39))
     (stroke (width 0) (type default))
   )
@@
     (stroke (width 0) (type default))
   )
-  (wire (pts (xy 146.05 72.39) (xy 147.32 72.39))
+  (wire (pts (xy 142.24 72.39) (xy 147.32 72.39))
     (stroke (width 0) (type default))
   )
-  (global_label "+BATT" (shape input) (at 146.05 72.39 180) (fields_autoplaced)
-    (effects (font (size 1.27 1.27)) (justify right))
-    (property "Intersheetrefs" "${INTERSHEET_REFS}" (at 137.1986 72.39 0)
-      (effects (font (size 1.27 1.27)) (justify right) hide)
-    )
-  )
-  (hierarchical_label "EXTERNAT_UART_TX" (shape output) (at 119.38 80.01 180) (fields_autoplaced)
+  (hierarchical_label "EXT_UART_TX" (shape output) (at 119.38 80.01 180) (fields_autoplaced)
     (effects (font (size 1.27 1.27)) (justify right))
   )
-  (hierarchical_label "EXTERNAL_UART_RX" (shape input) (at 120.65 86.36 180) (fields_autoplaced)
+  (hierarchical_label "EXT_UART_RX" (shape input) (at 120.65 86.36 180) (fields_autoplaced)
     (effects (font (size 1.27 1.27)) (justify right))
   )
   (symbol (lib_id "Device:R") (at 134.62 77.47 270) (unit 1)
     (in_bom yes) (on_board yes) (dnp no)
-    (property "Reference" "R20" (at 134.62 72.39 90)
+    (property "Reference" "R19" (at 134.62 72.39 90)
       (effects (font (size 1.27 1.27)))
     )
@@
       (effects (font (size 1.27 1.27)))
     )
-    (property "Footprint" "" (at 134.62 75.692 90)
+    (property "Footprint" "Resistor_SMD:R_0603_1608Metric" (at 134.62 75.692 90)
       (effects (font (size 1.27 1.27)) hide)
     )
@@
       (project "minimouse"
         (path "/d8fa4cba-2469-4231-847f-065b6b829f44/d17bb1c7-f68a-465e-9a17-5858ef86fc30"
-          (reference "R20") (unit 1)
+          (reference "R19") (unit 1)
         )
       )
@@
   (symbol (lib_id "Device:C") (at 217.17 36.83 180) (unit 1)
     (in_bom yes) (on_board yes) (dnp no) (fields_autoplaced)
-    (property "Reference" "C11" (at 220.98 35.56 0)
+    (property "Reference" "C14" (at 220.98 35.56 0)
       (effects (font (size 1.27 1.27)) (justify right))
     )
-    (property "Value" "C" (at 220.98 38.1 0)
+    (property "Value" "2.2uF" (at 220.98 38.1 0)
       (effects (font (size 1.27 1.27)) (justify right))
     )
-    (property "Footprint" "" (at 216.2048 33.02 0)
+    (property "Footprint" "Capacitor_SMD:C_0603_1608Metric" (at 216.2048 33.02 0)
       (effects (font (size 1.27 1.27)) hide)
     )
@@
       (project "minimouse"
         (path "/d8fa4cba-2469-4231-847f-065b6b829f44/d17bb1c7-f68a-465e-9a17-5858ef86fc30"
-          (reference "C11") (unit 1)
+          (reference "C14") (unit 1)
         )
       )
@@
   (symbol (lib_id "power:GND") (at 189.23 71.12 0) (unit 1)
     (in_bom yes) (on_board yes) (dnp no) (fields_autoplaced)
-    (property "Reference" "#PWR023" (at 189.23 77.47 0)
+    (property "Reference" "#PWR031" (at 189.23 77.47 0)
       (effects (font (size 1.27 1.27)) hide)
     )
@@
       (project "minimouse"
         (path "/d8fa4cba-2469-4231-847f-065b6b829f44/d17bb1c7-f68a-465e-9a17-5858ef86fc30"
-          (reference "#PWR023") (unit 1)
+          (reference "#PWR031") (unit 1)
         )
       )
@@
   (symbol (lib_id "Connector_Generic:Conn_01x04") (at 152.4 72.39 0) (unit 1)
     (in_bom yes) (on_board yes) (dnp no) (fields_autoplaced)
-    (property "Reference" "J4" (at 154.94 72.39 0)
+    (property "Reference" "J5" (at 154.94 72.39 0)
       (effects (font (size 1.27 1.27)) (justify left))
     )
@@
       (effects (font (size 1.27 1.27)) (justify left))
     )
-    (property "Footprint" "" (at 152.4 72.39 0)
+    (property "Footprint" "Connector_PinHeader_2.54mm:PinHeader_1x04_P2.54mm_Vertical" (at 152.4 72.39 0)
       (effects (font (size 1.27 1.27)) hide)
     )
@@
       (project "minimouse"
         (path "/d8fa4cba-2469-4231-847f-065b6b829f44/d17bb1c7-f68a-465e-9a17-5858ef86fc30"
-          (reference "J4") (unit 1)
+          (reference "J5") (unit 1)
         )
       )
@@
   (symbol (lib_id "power:+BATT") (at 217.17 25.4 0) (unit 1)
     (in_bom yes) (on_board yes) (dnp no) (fields_autoplaced)
-    (property "Reference" "#PWR025" (at 217.17 29.21 0)
+    (property "Reference" "#PWR032" (at 217.17 29.21 0)
       (effects (font (size 1.27 1.27)) hide)
     )
@@
       (project "minimouse"
         (path "/d8fa4cba-2469-4231-847f-065b6b829f44/d17bb1c7-f68a-465e-9a17-5858ef86fc30"
-          (reference "#PWR025") (unit 1)
+          (reference "#PWR032") (unit 1)
         )
       )
@@
   (symbol (lib_id "power:GND") (at 217.17 45.72 0) (unit 1)
     (in_bom yes) (on_board yes) (dnp no) (fields_autoplaced)
-    (property "Reference" "#PWR026" (at 217.17 52.07 0)
+    (property "Reference" "#PWR033" (at 217.17 52.07 0)
       (effects (font (size 1.27 1.27)) hide)
     )
@@
       (project "minimouse"
         (path "/d8fa4cba-2469-4231-847f-065b6b829f44/d17bb1c7-f68a-465e-9a17-5858ef86fc30"
-          (reference "#PWR026") (unit 1)
+          (reference "#PWR033") (unit 1)
         )
       )
+    )
+  )
+  (symbol (lib_id "power:+BATT") (at 142.24 64.77 0) (unit 1)
+    (in_bom yes) (on_board yes) (dnp no) (fields_autoplaced)
+    (property "Reference" "#PWR030" (at 142.24 68.58 0)
+      (effects (font (size 1.27 1.27)) hide)
+    )
+    (property "Value" "+BATT" (at 142.24 59.69 0)
+      (effects (font (size 1.27 1.27)))
+    )
+    (property "Footprint" "" (at 142.24 64.77 0)
+      (effects (font (size 1.27 1.27)) hide)
+    )
+    (property "Datasheet" "" (at 142.24 64.77 0)
+      (effects (font (size 1.27 1.27)) hide)
+    )
+    (pin "1")
+    (instances
+      (project "minimouse"
+        (path "/d8fa4cba-2469-4231-847f-065b6b829f44/d17bb1c7-f68a-465e-9a17-5858ef86fc30"
+          (reference "#PWR030") (unit 1)
+        )
+      )
