File: mm_mcu.kicad_sch (KiCad schematic)
At the start: 18 parts, among them J1 Conn_ARM_JTAG_SWD_10, U1 STM32F030C8Tx

Commit message: Pistes
Parts:
- removed R7: 100, Resistor_SMD:R_0603_1608Metric, symbol Device:R
- renumbered BOOT0 to BOOT1, C6 to C3, C1 to C4, C2 to C5, C3 to C6, C4 to C7, C5 to C8, J1 to J2, R1 to R2, R6 to R3, R8 to R4, R9 to R5, R2 to R6, R3 to R7, R4 to R8, R5 to R9, U1 to U2
Connections:
- net OUT_B1: now also U2.19 (PB1)
