File: mm_motor.kicad_sch (KiCad schematic)
At the start: 1 part, among them M1 N20_encoder

Commit message: fin TP2
Parts:
- added C12: 2.2uF, symbol Device:C
- added J2: Conn_01x06_Pin, symbol Connector:Conn_01x06_Pin
- added R16, R18: 100Ω, symbol Device:R
Connections:
- net C1: now also J2.3 (Pin_3)
- net C2: now also J2.4 (Pin_4)
- net MA: now also R16.2
- net MB: now also R18.2
- new net: J2.1 (Pin_1), R16.1
- new net: J2.6 (Pin_6), R18.1
- new net +BATT: C12.1, J2.5 (Pin_5)
- new net GND: C12.2, J2.2 (Pin_2)
Other:
- moved on the sheet: M1

Commit message: fin TP2 2
Changed lines of the file:
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@@
     (stroke (width 0) (type default))
   )
-  (wire (pts (xy 134.62 88.9) (xy 151.13 88.9))
+  (wire (pts (xy 134.62 88.9) (xy 181.61 88.9))
     (stroke (width 0) (type default))
   )
@@
     )
   )
-  (symbol (lib_id "power:GND") (at 151.13 88.9 0) (unit 1)
-    (in_bom yes) (on_board yes) (dnp no) (fields_autoplaced)
-    (property "Reference" "#PWR08" (at 151.13 95.25 0)
-      (effects (font (size 1.27 1.27)) hide)
-    )
-    (property "Value" "GND" (at 151.13 93.98 0)
-      (effects (font (size 1.27 1.27)))
-    )
-    (property "Footprint" "" (at 151.13 88.9 0)
-      (effects (font (size 1.27 1.27)) hide)
-    )
-    (property "Datasheet" "" (at 151.13 88.9 0)
-      (effects (font (size 1.27 1.27)) hide)
-    )
+  (symbol (lib_id "power:GND") (at 181.61 88.9 0) (unit 1)
+    (in_bom yes) (on_board yes) (dnp no) (fields_autoplaced)
+    (property "Reference" "#PWR08" (at 181.61 95.25 0)
+      (effects (font (size 1.27 1.27)) hide)
+    )
+    (property "Value" "GND" (at 181.61 93.98 0)
+      (effects (font (size 1.27 1.27)))
+    )
+    (property "Footprint" "" (at 181.61 88.9 0)
+      (effects (font (size 1.27 1.27)) hide)
+    )
+    (property "Datasheet" "" (at 181.61 88.9 0)
+      (effects (font (size 1.27 1.27)) hide)
+    )

Commit message: Pistes
Parts:
- C12: footprint (none) -> Capacitor_SMD:C_0603_1608Metric
- J3: renamed from J2; footprint (none) -> Connector_PinHeader_2.54mm:PinHeader_1x06_P2.54mm_Vertical
- R15: renamed from R18; footprint (none) -> Resistor_SMD:R_0603_1608Metric
- R16: footprint (none) -> Resistor_SMD:R_0603_1608Metric
Connections:
- net C1: now also R16.2; no longer J3.3 (Pin_3)
- net C2: now also R15.2; no longer J3.4 (Pin_4)
- net MA: now also J3.1 (Pin_1); no longer R16.2
- net MB: now also J3.6 (Pin_6); no longer R15.2
- net at R16.1: now also J3.3 (Pin_3); no longer J3.1 (Pin_1)
- net at R15.1: now also J3.4 (Pin_4); no longer J3.6 (Pin_6)
Other:
- moved on the sheet: R15, R16
