File: minimouse.kicad_pcb (KiCad board)
At the start: 2 copper layers, 90 x 85 mm, 22 parts, among them J1 Conn_ARM_JTAG_SWD_10, J5 Conn_01x02, M1 N20_encoder, M2 N20_encoder, U1 STM32F030C8Tx, U4 HC-SR04

Commit message: Pistes
Parts:
- removed BOOT0: TestPoint, TestPoint:TestPoint_Pad_D1.5mm
- added BOOT1: TestPoint, TestPoint:TestPoint_Pad_D1.5mm, F.Cu at (153.4, 129.8)
- added C10: 22nF, Capacitor_SMD:C_0603_1608Metric, F.Cu at (127.0, 70.4)
- added C11: 2.2uF, Capacitor_SMD:C_0603_1608Metric, F.Cu at (140.7, 113.8)
- added C12: 2.2uF, Capacitor_SMD:C_0603_1608Metric, F.Cu at (178.1, 114.6)
- added C13: 2.2uF, Capacitor_SMD:C_0603_1608Metric, F.Cu at (177.8, 119.4)
- added C14: 2.2uF, Capacitor_SMD:C_0603_1608Metric, B.Cu at (159.5, 119.5)
- added C15: 2.2uF, Capacitor_SMD:C_0603_1608Metric, F.Cu at (143.1, 90.9)
- added C7: 0.1uF, Capacitor_SMD:C_0603_1608Metric, F.Cu at (116.3, 80.3)
- added C8: 0.1uF, Capacitor_SMD:C_0603_1608Metric, F.Cu at (116.3, 77.0)
- added C9: 1nF, Capacitor_SMD:C_0603_1608Metric, F.Cu at (156.7, 75.9)
- added D1: LED, LED_SMD:LED_0603_1608Metric, F.Cu at (176.8, 95.1)
- added J2: Conn_ARM_JTAG_SWD_10, Connector_PinHeader_1.27mm:PinHeader_2x05_P1.27mm_Vertical, F.Cu at (148.6, 135.6)
- added J3: Conn_01x06_Pin, Connector_PinHeader_2.54mm:PinHeader_1x06_P2.54mm_Vertical, F.Cu at (174.0, 85.3)
- added J4: Conn_01x06_Pin, Connector_PinHeader_2.54mm:PinHeader_1x06_P2.54mm_Vertical, F.Cu at (132.2, 91.9)
- added R10: 10kΩ, Resistor_SMD:R_0603_1608Metric, F.Cu at (145.2, 98.2)
- added R11: 10kΩ, Resistor_SMD:R_0603_1608Metric, F.Cu at (160.2, 107.8)
- added R12: 10kΩ, Resistor_SMD:R_0603_1608Metric, F.Cu at (145.5, 79.8)
- added R13: 1kΩ, Resistor_SMD:R_0603_1608Metric, F.Cu at (129.3, 75.7)
- added R14: 47kΩ, Resistor_SMD:R_0603_1608Metric, F.Cu at (125.5, 75.7)
- added R16: 100Ω, Resistor_SMD:R_0603_1608Metric, F.Cu at (164.1, 78.2)
- added R17: 100Ω, Resistor_SMD:R_0603_1608Metric, F.Cu at (134.2, 85.7)
- added R18: 100Ω, Resistor_SMD:R_0603_1608Metric, F.Cu at (139.9, 91.6)
- added R19: 100Ω, Resistor_SMD:R_0603_1608Metric, F.Cu at (152.7, 76.5)
- added R20: 100, Resistor_SMD:R_0603_1608Metric, F.Cu at (160.0, 72.4)
- added RSENSE1: 330mΩ, Resistor_SMD:R_2512_6332Metric, F.Cu at (154.2, 107.8)
- added RSENSE2: 330mΩ, Resistor_SMD:R_2512_6332Metric, F.Cu at (161.4, 101.3)
- added U2: STM32F030C8Tx, Package_QFP:LQFP-48_7x7mm_P0.5mm, F.Cu at (152.0, 84.0)
- added U3: STSPIN240, Package_DFN_QFN:VQFN-16-1EP_3x3mm_P0.5mm_EP1.8x1.8mm, F.Cu at (151.3, 97.6)
- added locked: 100Ω, Resistor_SMD:R_0603_1608Metric, F.Cu at (163.8, 74.2)
- C2, C3, C4: value 0.1uF -> 2.2uF
- C6: value 2.2uF -> 0.1uF
- J1: value Conn_ARM_JTAG_SWD_10 -> Conn_01x02; footprint Connector_PinHeader_1.27mm:PinHeader_2x05_P1.27mm_Vertical -> Connector_PinHeader_2.54mm:PinHeader_1x02_P2.54mm_Vertical
- J5: value Conn_01x02 -> Conn_01x04; footprint Connector_PinHeader_2.54mm:PinHeader_1x02_P2.54mm_Vertical -> Connector_PinHeader_2.54mm:PinHeader_1x04_P2.54mm_Vertical
- R1: value 10k -> 330
- R2: value 100 -> 10k
- U1: value STM32F030C8Tx -> LP5907MFX-3.3; footprint Package_QFP:LQFP-48_7x7mm_P0.5mm -> Package_TO_SOT_SMD:SOT-23-5
- moved J5 51.9 mm to (164.6, 84.6), turned to 0 degrees
- moved C1 48.9 mm to (190.4, 94.8), turned to 0 degrees
- moved C4 40.0 mm to (116.3, 92.5)
- moved C2 35.3 mm to (179.8, 89.3), turned to 0 degrees
- moved U1 32.6 mm to (181.7, 96.1)
- moved R2 32.4 mm to (148.5, 127.3), turned to 180 degrees
- moved R4 29.6 mm to (145.3, 129.0), turned to 0 degrees
- moved C3 27.9 mm to (116.4, 96.5), turned to 0 degrees
- moved C6 27.3 mm to (116.3, 84.6), turned to 0 degrees
- moved R1 26.9 mm to (172.7, 94.4), turned to 0 degrees
- moved R5 23.4 mm to (146.7, 76.1), turned to 180 degrees
- moved J1 20.8 mm to (184.7, 84.0), turned to 90 degrees
- moved R3 16.7 mm to (157.9, 91.9), turned to 90 degrees
- moved R9 13.3 mm to (154.9, 91.8)
- moved R8 10.9 mm to (152.6, 91.8)
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Connections:
- C1 pad 1: +3.3V -> +BATT
- J1 pad 1: +3.3V -> GND
- J1 pad 2: /mcu/SWDIO -> +BATT
- R1 pad 1: /mcu/BOOT0 -> +3.3V
- R1 pad 2: GND -> Net-(D1-A)
- R2 pad 1: Net-(U1-PA2) -> /mcu/BOOT0
- R2 pad 2: /mcu/TIM15_CH1 -> GND
- R3 pad 1: Net-(U1-PA3) -> /mcu/OUT_B0
- R3 pad 2: /mcu/TIM15_CH2 -> Net-(U2-PB0)
- R4 pad 1: Net-(U1-PA4) -> /external_uart/EXT_UART_RX
- R4 pad 2: /mcu/OUT_A4 -> Net-(U2-PB6)
- R5 pad 1: Net-(U1-PA5) -> /mcu/OUT_B9
- R5 pad 2: /mcu/OUT_A5 -> Net-(U2-PB9)
- R6 pad 1: /mcu/OUT_B0 -> Net-(U2-PA2)
- R6 pad 2: Net-(U1-PB0) -> /mcu/TIM15_CH1
- R7 pad 1: /mcu/OUT_B1 -> Net-(U2-PA3)
- R7 pad 2: Net-(U1-PB1) -> /mcu/TIM15_CH2
- R8 pad 1: /mcu/UART1_TX -> Net-(U2-PA4)
- R8 pad 2: Net-(U1-PB6) -> /mcu/OUT_A4
- R9 pad 1: /mcu/OUT_B9 -> Net-(U2-PA5)
- R9 pad 2: Net-(U1-PB9) -> /mcu/OUT_A5
- U1 pad 1: +3.3V -> +BATT
- U1 pad 2: unconnected-(U1-PC13-Pad2) -> GND
- U1 pad 3: unconnected-(U1-PC14-Pad3) -> +BATT
- U1 pad 5: unconnected-(U1-PF0-Pad5) -> +3.3V
- U4 pad 4: +3V3 -> +3.3V
Routing:
- net GND: track 0.00 -> 66.0 mm
- net +3.3V: track 0.00 -> 56.3 mm
- net +BATT: track 0.00 -> 24.4 mm
- net /mcu/TIM15_CH2: track 0.00 -> 8.60 mm
- net Net-(U2-PB0): track 0.00 -> 7.93 mm
- net /mcu/OUT_B0: track 0.00 -> 7.42 mm
- net Net-(C10-Pad1): track 0.00 -> 7.04 mm
- net /mcu/TIM15_CH1: track 0.00 -> 6.69 mm
- net Net-(U2-PA5): track 0.00 -> 6.34 mm
- net /mcu/OUT_A5: track 0.00 -> 5.75 mm
- net Net-(U2-PA4): track 0.00 -> 4.46 mm
- net Net-(U2-PA2): track 0.00 -> 4.01 mm
- net /mcu/OUT_A4: track 0.00 -> 3.64 mm
- net Net-(D1-A): track 0.00 -> 3.21 mm
- net Net-(U2-PA3): track 0.00 -> 2.92 mm
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
Commit message: PCB2
Parts:
- U2: value STM32F030C8Tx -> locked
- moved C13 66.2 mm to (121.2, 85.0), turned to 90 degrees
- moved J2 58.3 mm to (160.2, 78.5), turned to -90 degrees
- moved C14 51.9 mm to (133.7, 74.5), turned to -90 degrees
- moved BOOT1 49.3 mm to (150.5, 80.6)
- moved R2 49.3 mm to (150.6, 78.0), turned to 0 degrees
- moved C10 47.2 mm to (162.2, 101.9), turned to 90 degrees
- moved R4 44.9 mm to (144.8, 84.1), turned to -90 degrees
- moved C8 43.9 mm to (158.2, 90.1)
- moved R14 42.7 mm to (159.7, 101.1), turned to 0 degrees
- moved C7 42.5 mm to (158.3, 87.2)
- moved C6 42.0 mm to (158.3, 83.8), turned to 180 degrees
- moved R13 40.7 mm to (159.7, 102.7)
- moved C5 40.4 mm to (156.4, 93.7)
- moved C4 32.1 mm to (146.7, 82.1), turned to 90 degrees
- moved C3 29.4 mm to (144.7, 88.8), turned to 90 degrees
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Routing:
- net +BATT: track 24.4 -> 95.4 mm
- net /external_uart/EXT_UART_TX: track 0.00 -> 45.1 mm, vias 0 -> 2
- net /mcu/SWDIO: track 0.00 -> 40.0 mm
- net /mcu/~{RESET}: track 0.00 -> 40.0 mm
- net /motorB/MB: track 0.00 -> 39.6 mm
- net /motorA/MB: track 0.00 -> 35.6 mm, vias 0 -> 2
- net /motorA/MA: track 0.00 -> 33.6 mm
- net /mcu/TIM2_CH2: track 0.00 -> 26.9 mm
- net /mcu/TIM3_CH1: track 0.00 -> 26.2 mm
- net /mcu/TIM2_CH1: track 0.00 -> 24.1 mm
- net /motorB/MA: track 0.00 -> 23.2 mm
- net /mcu/TIM3_CH2: track 0.00 -> 22.2 mm
- net Net-(U2-PB6): track 0.00 -> 19.9 mm, vias 0 -> 2
- net +3.3V: track 56.3 -> 75.4 mm, vias 0 -> 2
- net /mcu/OUT_B1: track 0.00 -> 12.3 mm
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
Commit message: lastmodif
Parts:
- added D2: 1.5KExxA, Diode_THT:D_DO-201AE_P15.24mm_Horizontal, F.Cu at (136.8, 102.5)
- added Q1: PMOS, Package_TO_SOT_SMD:SOT-23-3, F.Cu at (127.0, 97.5)
- added R21: 100, Resistor_SMD:R_0603_1608Metric, F.Cu at (123.7, 97.3)
- added R22: 10K, Resistor_SMD:R_0603_1608Metric, F.Cu at (130.6, 97.4)
- added TP1: TestPoint, TestPoint:TestPoint_Pad_D1.5mm, F.Cu at (120.1, 96.5)
- added TP2: TestPoint, TestPoint:TestPoint_Pad_D1.5mm, F.Cu at (114.7, 96.1)
- added TP3: TestPoint, TestPoint:TestPoint_Pad_D1.5mm, F.Cu at (136.2, 96.2)
- C14: moved to F.Cu
- moved C7 13.8 mm to (144.6, 85.5), turned to -90 degrees
- moved RSENSE1 12.2 mm to (162.3, 109.6), turned to -90 degrees
- moved J3 10.6 mm to (167.9, 89.9), turned to 90 degrees
- moved R4 9.69 mm to (153.2, 79.1)
- moved C10 5.96 mm to (165.4, 96.9)
- moved R13 5.96 mm to (163.0, 97.7)
- moved R14 5.96 mm to (163.0, 96.1)
- moved C13 2.33 mm to (120.4, 87.2), turned to 180 degrees
- moved R2 1.39 mm to (150.5, 76.7), turned to 90 degrees
- moved C6 1.00 mm to (157.3, 83.6), turned to 90 degrees
- moved RSENSE2 0.53 mm to (144.2, 105.8)
Connections:
- U4 pad 4: +3.3V -> +BATT
Routing:
- net +BATT: track 95.4 -> 183.3 mm, vias 0 -> 3
- net /mcu/SWDIO: track 40.0 -> 10.6 mm, vias 0 -> 1
- net /external_uart/EXT_UART_TX: track 45.1 -> 16.0 mm
- net /mcu/~{RESET}: track 40.0 -> 12.3 mm, vias 0 -> 1
- net GND: track 73.8 -> 48.5 mm, vias 0 -> 39
- net +3.3V: track 75.4 -> 99.9 mm
- net Net-(U2-PB6): track 19.9 -> 4.63 mm, vias 2 -> 0
- net Net-(D2-A1): track 0.00 -> 10.7 mm
- net /external_uart/EXT_UART_RX: track 7.89 -> 18.0 mm, vias 0 -> 2
- net Net-(D2-A2): track 0.00 -> 7.61 mm
- net /motorA/MB: track 35.6 -> 40.9 mm, vias 2 -> 0
- net /mcu/TIM3_CH1: track 26.2 -> 21.6 mm, vias 0 -> 2
- net Net-(J3-Pin_4): track 11.0 -> 6.42 mm
- net /motorA/MA: track 33.6 -> 30.9 mm
- net /mcu/TIM3_CH2: track 22.2 -> 24.8 mm, vias 0 -> 2
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- added copper zone on B.Cu, net GND
- added copper zone on F.Cu, net GND
