File: mm_power.kicad_sch (KiCad schematic)
At the start: 1 part, among them J5 Conn_01x02

Commit message: fin TP2
Parts:
- added U3: LP5907MFX-3.3, Package_TO_SOT_SMD:SOT-23-5, symbol Regulator_Linear:LP5907MFX-3.3
Changed lines of the file:
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@@
     (stroke (width 0) (type default))
+  )
+  (symbol (lib_id "Regulator_Linear:LP5907MFX-3.3") (at 115.57 67.31 0) (unit 1)
+    (in_bom yes) (on_board yes) (dnp no) (fields_autoplaced)
+    (property "Reference" "U3" (at 115.57 57.15 0)
+      (effects (font (size 1.27 1.27)))
+    )
+    (property "Value" "LP5907MFX-3.3" (at 115.57 59.69 0)
+      (effects (font (size 1.27 1.27)))
+    )
+    (property "Footprint" "Package_TO_SOT_SMD:SOT-23-5" (at 115.57 58.42 0)
+      (effects (font (size 1.27 1.27)) hide)
+    )
+    (property "Datasheet" "http://www.ti.com/lit/ds/symlink/lp5907.pdf" (at 115.57 54.61 0)
+      (effects (font (size 1.27 1.27)) hide)
+    )
+    (pin "2")
+    (pin "3")
+    (pin "1")
+    (pin "5")
+    (pin "4")
+    (instances
+      (project "minimouse"
+        (path "/d8fa4cba-2469-4231-847f-065b6b829f44/3f9b0845-5778-418c-a7a8-03da2392145e"
+          (reference "U3") (unit 1)
+        )
+      )
+    )
   )
   (symbol (lib_id "power:+BATT") (at 86.36 74.93 0) (unit 1)

Commit message: fin TP2 2
Parts:
- added C14: 1uF, Capacitor_SMD:C_0603_1608Metric, symbol Device:C
- added C15: 1uF, symbol Device:C
Connections:
- net +BATT: now also U3.1 (IN), C14.1
- net GND: now also U3.2 (GND), C14.2, C15.2
- net +3.3V: now reaches U3.5 (OUT)
- net +3.3V: now also C15.1
Other:
- moved on the sheet: U3
Changed lines of the file:
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@@
   (junction (at 86.36 82.55) (diameter 0) (color 0 0 0 0)
   )
+  (junction (at 128.27 49.53) (diameter 0) (color 0 0 0 0)
+  )
   (junction (at 86.36 95.25) (diameter 0) (color 0 0 0 0)
   )
+  (junction (at 157.48 49.53) (diameter 0) (color 0 0 0 0)
+  )
   (wire (pts (xy 86.36 90.17) (xy 86.36 95.25))
     (stroke (width 0) (type default))
   )
+  (wire (pts (xy 128.27 49.53) (xy 128.27 46.99))
+    (stroke (width 0) (type default))
+  )
   (wire (pts (xy 95.25 82.55) (xy 86.36 82.55))
     (stroke (width 0) (type default))
@@
     (stroke (width 0) (type default))
   )
+  (wire (pts (xy 138.43 49.53) (xy 128.27 49.53))
+    (stroke (width 0) (type default))
+  )
+  (wire (pts (xy 157.48 49.53) (xy 162.56 49.53))
+    (stroke (width 0) (type default))
+  )
   (wire (pts (xy 80.01 87.63) (xy 86.36 87.63))
     (stroke (width 0) (type default))
   )
+  (wire (pts (xy 153.67 49.53) (xy 157.48 49.53))
+    (stroke (width 0) (type default))
+  )
   (wire (pts (xy 86.36 95.25) (xy 86.36 100.33))
     (stroke (width 0) (type default))
@@
     (stroke (width 0) (type default))
   )
+  (wire (pts (xy 128.27 49.53) (xy 128.27 50.8))
+    (stroke (width 0) (type default))
+  )
+  (wire (pts (xy 128.27 58.42) (xy 128.27 60.96))
+    (stroke (width 0) (type default))
+  )
   (wire (pts (xy 80.01 90.17) (xy 86.36 90.17))
     (stroke (width 0) (type default))
   )
-  (symbol (lib_id "Regulator_Linear:LP5907MFX-3.3") (at 115.57 67.31 0) (unit 1)
-    (in_bom yes) (on_board yes) (dnp no) (fields_autoplaced)
-    (property "Reference" "U3" (at 115.57 57.15 0)
-      (effects (font (size 1.27 1.27)))
-    )
-    (property "Value" "LP5907MFX-3.3" (at 115.57 59.69 0)
-      (effects (font (size 1.27 1.27)))
-    )
-    (property "Footprint" "Package_TO_SOT_SMD:SOT-23-5" (at 115.57 58.42 0)
-      (effects (font (size 1.27 1.27)) hide)
-    )
-    (property "Datasheet" "http://www.ti.com/lit/ds/symlink/lp5907.pdf" (at 115.57 54.61 0)
+  (symbol (lib_id "power:+BATT") (at 128.27 46.99 0) (unit 1)
+    (in_bom yes) (on_board yes) (dnp no) (fields_autoplaced)
+    (property "Reference" "#PWR031" (at 128.27 50.8 0)
+      (effects (font (size 1.27 1.27)) hide)
+    )
+    (property "Value" "+BATT" (at 128.27 41.91 0)
+      (effects (font (size 1.27 1.27)))
+    )
+    (property "Footprint" "" (at 128.27 46.99 0)
+      (effects (font (size 1.27 1.27)) hide)
+    )
+    (property "Datasheet" "" (at 128.27 46.99 0)
+      (effects (font (size 1.27 1.27)) hide)
+    )
+    (pin "1")
+    (instances
+      (project "minimouse"
+        (path "/d8fa4cba-2469-4231-847f-065b6b829f44/3f9b0845-5778-418c-a7a8-03da2392145e"
+          (reference "#PWR031") (unit 1)
+        )
+      )
+    )
+  )
+  (symbol (lib_id "Regulator_Linear:LP5907MFX-3.3") (at 146.05 52.07 0) (unit 1)
+    (in_bom yes) (on_board yes) (dnp no) (fields_autoplaced)
+    (property "Reference" "U3" (at 146.05 41.91 0)
+      (effects (font (size 1.27 1.27)))
+    )
+    (property "Value" "LP5907MFX-3.3" (at 146.05 44.45 0)
+      (effects (font (size 1.27 1.27)))
+    )
+    (property "Footprint" "Package_TO_SOT_SMD:SOT-23-5" (at 146.05 43.18 0)
+      (effects (font (size 1.27 1.27)) hide)
+    )
+    (property "Datasheet" "http://www.ti.com/lit/ds/symlink/lp5907.pdf" (at 146.05 39.37 0)
       (effects (font (size 1.27 1.27)) hide)
     )
@@
         )
       )
+    )
+  )
+  (symbol (lib_id "power:GND") (at 146.05 59.69 0) (unit 1)
+    (in_bom yes) (on_board yes) (dnp no) (fields_autoplaced)
+    (property "Reference" "#PWR024" (at 146.05 66.04 0)
+      (effects (font (size 1.27 1.27)) hide)
+    )
+    (property "Value" "GND" (at 146.05 64.77 0)
+      (effects (font (size 1.27 1.27)))
+    )
+    (property "Footprint" "" (at 146.05 59.69 0)
+      (effects (font (size 1.27 1.27)) hide)
+    )
+    (property "Datasheet" "" (at 146.05 59.69 0)
+      (effects (font (size 1.27 1.27)) hide)
+    )
+    (pin "1")
+    (instances
+      (project "minimouse"
+        (path "/d8fa4cba-2469-4231-847f-065b6b829f44/3f9b0845-5778-418c-a7a8-03da2392145e"
+          (reference "#PWR024") (unit 1)
+        )
+      )
+    )
+  )
+  (symbol (lib_id "Device:C") (at 128.27 54.61 0) (unit 1)
+    (in_bom yes) (on_board yes) (dnp no) (fields_autoplaced)
+    (property "Reference" "C14" (at 132.08 53.34 0)
+      (effects (font (size 1.27 1.27)) (justify left))
+    )
+    (property "Value" "1uF" (at 132.08 55.88 0)
+      (effects (font (size 1.27 1.27)) (justify left))
+    )
+    (property "Footprint" "Capacitor_SMD:C_0603_1608Metric" (at 129.2352 58.42 0)
+      (effects (font (size 1.27 1.27)) hide)
+    )
+    (property "Datasheet" "~" (at 128.27 54.61 0)
+      (effects (font (size 1.27 1.27)) hide)
+    )
+    (pin "1")
+    (pin "2")
+    (instances
+      (project "minimouse"
+        (path "/d8fa4cba-2469-4231-847f-065b6b829f44/3f9b0845-5778-418c-a7a8-03da2392145e"
+          (reference "C14") (unit 1)
+        )
+      )
+    )
+  )
+  (symbol (lib_id "power:GND") (at 128.27 60.96 0) (unit 1)
+    (in_bom yes) (on_board yes) (dnp no) (fields_autoplaced)
+    (property "Reference" "#PWR029" (at 128.27 67.31 0)
+      (effects (font (size 1.27 1.27)) hide)
+    )
+    (property "Value" "GND" (at 128.27 66.04 0)
+      (effects (font (size 1.27 1.27)))
+    )
+    (property "Footprint" "" (at 128.27 60.96 0)
+      (effects (font (size 1.27 1.27)) hide)
+    )
+    (property "Datasheet" "" (at 128.27 60.96 0)
+      (effects (font (size 1.27 1.27)) hide)
+    )
+    (pin "1")
+    (instances
+      (project "minimouse"
+        (path "/d8fa4cba-2469-4231-847f-065b6b829f44/3f9b0845-5778-418c-a7a8-03da2392145e"
+          (reference "#PWR029") (unit 1)
+        )
+      )
+    )
+  )
+  (symbol (lib_id "power:GND") (at 157.48 57.15 0) (unit 1)
+    (in_bom yes) (on_board yes) (dnp no) (fields_autoplaced)
+    (property "Reference" "#PWR030" (at 157.48 63.5 0)
+      (effects (font (size 1.27 1.27)) hide)
+    )
+    (property "Value" "GND" (at 157.48 62.23 0)
+      (effects (font (size 1.27 1.27)))
+    )
+    (property "Footprint" "" (at 157.48 57.15 0)
+      (effects (font (size 1.27 1.27)) hide)
+    )
+    (property "Datasheet" "" (at 157.48 57.15 0)
+      (effects (font (size 1.27 1.27)) hide)
+    )
+    (pin "1")
+    (instances
+      (project "minimouse"
+        (path "/d8fa4cba-2469-4231-847f-065b6b829f44/3f9b0845-5778-418c-a7a8-03da2392145e"
+          (reference "#PWR030") (unit 1)
+        )
+      )
+    )
+  )
+  (symbol (lib_id "power:+3.3V") (at 162.56 49.53 0) (unit 1)
+    (in_bom yes) (on_board yes) (dnp no) (fields_autoplaced)
+    (property "Reference" "#PWR032" (at 162.56 53.34 0)
+      (effects (font (size 1.27 1.27)) hide)
+    )
+    (property "Value" "+3.3V" (at 162.56 44.45 0)
+      (effects (font (size 1.27 1.27)))
+    )
+    (property "Footprint" "" (at 162.56 49.53 0)
+      (effects (font (size 1.27 1.27)) hide)
+    )
+    (property "Datasheet" "" (at 162.56 49.53 0)
+      (effects (font (size 1.27 1.27)) hide)
+    )
+    (pin "1")
+    (instances
+      (project "minimouse"
+        (path "/d8fa4cba-2469-4231-847f-065b6b829f44/3f9b0845-5778-418c-a7a8-03da2392145e"
+          (reference "#PWR032") (unit 1)
+        )
+      )
+    )
+  )
+  (symbol (lib_id "Device:C") (at 157.48 53.34 0) (unit 1)
+    (in_bom yes) (on_board yes) (dnp no) (fields_autoplaced)
+    (property "Reference" "C15" (at 161.29 52.07 0)
+      (effects (font (size 1.27 1.27)) (justify left))
+    )
+    (property "Value" "1uF" (at 161.29 54.61 0)
+      (effects (font (size 1.27 1.27)) (justify left))
+    )
+    (property "Footprint" "" (at 158.4452 57.15 0)
+      (effects (font (size 1.27 1.27)) hide)
+    )
+    (property "Datasheet" "~" (at 157.48 53.34 0)
+      (effects (font (size 1.27 1.27)) hide)
+    )
+    (pin "1")
+    (pin "2")
+    (instances
+      (project "minimouse"
+        (path "/d8fa4cba-2469-4231-847f-065b6b829f44/3f9b0845-5778-418c-a7a8-03da2392145e"
+          (reference "C15") (unit 1)
+        )
+      )

Commit message: Pistes
Parts:
- added D1: LED, LED_SMD:LED_0603_1608Metric, symbol Device:LED
- added R1: 330, Resistor_SMD:R_0603_1608Metric, symbol Device:R
- C1: renamed from C14; value 1uF -> 2.2uF
- C2: renamed from C15; value 1uF -> 2.2uF; footprint (none) -> Capacitor_SMD:C_0603_1608Metric
- renumbered J5 to J1, U3 to U1
Connections:
- net +3.3V: now also R1.1
- net +BATT: now also U1.3 (EN)
- net GND: now also D1.1 (K)
- new net: D1.2 (A), R1.2

Commit message: lastmodif
Parts:
- added D2: 1.5KExxA, Diode_THT:D_DO-201AE_P15.24mm_Horizontal, symbol Diode:1.5KExxA
- added Q1: PMOS, Package_TO_SOT_SMD:SOT-23-3, symbol Simulation_SPICE:PMOS
- added R21: 100, Resistor_SMD:R_0603_1608Metric, symbol Device:R
- added R22: 10K, Resistor_SMD:R_0603_1608Metric, symbol Device:R
- added TP1, TP2, TP3: TestPoint, TestPoint:TestPoint_Pad_D1.5mm, symbol Connector:TestPoint
Connections:
- net +3.3V: now also TP3.1
- net +BATT: now also Q1.1 (D), R21.1, R22.1, TP1.1
- net GND: now also TP2.1
- new net: D2.2 (A2), Q1.2 (G), R21.2
- new net: D2.1 (A1), Q1.3 (S), R22.2
Other:
- moved on the sheet: J1
